File: hardware/kicad/MiniBurst/Power.kicad_sch (KiCad schematic)
At the start: 14 parts, among them J7 Conn_01x10_Pin, U1 LM358, U2 40106, U4 LM358, U5 LM358

Commit message: v0.1 PCB
Parts:
- J7: footprint Connector_IDC:IDC-Header_2x05_P2.54mm_Vertical -> benjiaomodular:Header_IDC2x05_NoArrow
Changed lines of the file:
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@@
 			)
 		)
-		(property "Footprint" "Connector_IDC:IDC-Header_2x05_P2.54mm_Vertical"
+		(property "Footprint" "benjiaomodular:Header_IDC2x05_NoArrow"
 			(at 36.83 66.04 0)
 			(effects
