File: hardware/legacy_versions/v0.1/kicad/MiniBurst/MiniBurst.kicad_sch (KiCad schematic)
At the start: 60 parts, among them J1 TRIG_IN, J2 TRIG_OUT, J3 EXT_CLK, J4 DURATION_OUT, J5 END_OUT, J6 PULSES_OUT, SW2 STEPS, SW3 SW_DPDT_x2, U1 LM358, U2 40106, U3 4017, U4 LM358, U5 LM358

Commit message: Adjusted main pcb dimensions to fit 3d printed rails
Parts:
- U1, U4, U5: footprint Package_SO:SOIC-8_5.23x5.23mm_P1.27mm -> Package_SO:SOIC-8_3.9x4.9mm_P1.27mm
- U3: footprint Package_SO:SOIC-16W_5.3x10.2mm_P1.27mm -> Package_SO:SOIC-16_3.9x9.9mm_P1.27mm; URL https://mou.sr/3BQ06Wp -> https://mou.sr/3zhJZjO
Changed lines of the file:
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@@
 	(title_block
 		(title "MiniBurst")
-		(rev "v0.2")
+		(rev "v0.1")
 		(company "benjiaomodular")
 	)
@@
 			)
 		)
-		(property "Footprint" "Package_SO:SOIC-8_5.23x5.23mm_P1.27mm"
+		(property "Footprint" "Package_SO:SOIC-8_3.9x4.9mm_P1.27mm"
 			(at 88.9 110.49 0)
 			(effects
@@
 			)
 		)
-		(property "Footprint" "Package_SO:SOIC-8_5.23x5.23mm_P1.27mm"
+		(property "Footprint" "Package_SO:SOIC-8_3.9x4.9mm_P1.27mm"
 			(at 146.05 20.32 0)
 			(effects
@@
 			)
 		)
-		(property "Footprint" "Package_SO:SOIC-8_5.23x5.23mm_P1.27mm"
+		(property "Footprint" "Package_SO:SOIC-8_3.9x4.9mm_P1.27mm"
 			(at 160.02 53.34 0)
 			(effects
@@
 			)
 		)
-		(property "Footprint" "Package_SO:SOIC-8_5.23x5.23mm_P1.27mm"
+		(property "Footprint" "Package_SO:SOIC-8_3.9x4.9mm_P1.27mm"
 			(at 77.47 31.75 0)
 			(effects
@@
 			)
 		)
-		(property "Footprint" "Package_SO:SOIC-8_5.23x5.23mm_P1.27mm"
+		(property "Footprint" "Package_SO:SOIC-8_3.9x4.9mm_P1.27mm"
 			(at 158.75 72.39 0)
 			(effects
@@
 			)
 		)
-		(property "Footprint" "Package_SO:SOIC-8_5.23x5.23mm_P1.27mm"
+		(property "Footprint" "Package_SO:SOIC-8_3.9x4.9mm_P1.27mm"
 			(at 133.35 137.16 0)
 			(effects
@@
 			)
 		)
-		(property "Footprint" "Package_SO:SOIC-16W_5.3x10.2mm_P1.27mm"
+		(property "Footprint" "Package_SO:SOIC-16_3.9x9.9mm_P1.27mm"
 			(at 222.25 132.08 0)
 			(effects
@@
 			)
 		)
-		(property "URL" "https://mou.sr/3BQ06Wp"
+		(property "URL" "https://mou.sr/3zhJZjO"
 			(at 222.25 132.08 0)
 			(effects
