File: hardware/legacy_versions/v0.1/kicad/MiniBurst/Power.kicad_sch (KiCad schematic)
At the start: 14 parts, among them J7 Conn_01x10_Pin, U1 LM358, U2 40106, U4 LM358, U5 LM358

Commit message: Adjusted main pcb dimensions to fit 3d printed rails
Parts:
- C3, C4: footprint Capacitor_SMD:CP_Elec_4x3.9 -> Capacitor_SMD:CP_Elec_6.3x4.5
- U1, U4, U5: footprint Package_SO:SOIC-8_5.23x5.23mm_P1.27mm -> Package_SO:SOIC-8_3.9x4.9mm_P1.27mm
Changed lines of the file:
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@@
 			)
 		)
-		(property "Footprint" "Capacitor_SMD:CP_Elec_4x3.9"
+		(property "Footprint" "Capacitor_SMD:CP_Elec_6.3x4.5"
 			(at 51.7652 73.66 0)
 			(effects
@@
 			)
 		)
-		(property "Footprint" "Capacitor_SMD:CP_Elec_4x3.9"
+		(property "Footprint" "Capacitor_SMD:CP_Elec_6.3x4.5"
 			(at 51.7652 63.5 0)
 			(effects
@@
 			)
 		)
-		(property "Footprint" "Package_SO:SOIC-8_5.23x5.23mm_P1.27mm"
+		(property "Footprint" "Package_SO:SOIC-8_3.9x4.9mm_P1.27mm"
 			(at 176.53 64.77 0)
 			(effects
@@
 			)
 		)
-		(property "Footprint" "Package_SO:SOIC-8_5.23x5.23mm_P1.27mm"
+		(property "Footprint" "Package_SO:SOIC-8_3.9x4.9mm_P1.27mm"
 			(at 151.13 64.77 0)
 			(effects
@@
 			)
 		)
-		(property "Footprint" "Package_SO:SOIC-8_5.23x5.23mm_P1.27mm"
+		(property "Footprint" "Package_SO:SOIC-8_3.9x4.9mm_P1.27mm"
 			(at 162.56 64.77 0)
 			(effects
